Commit message: Aggiunta simulazione del gripper su gazebo usando moveit

File: fmauch_universal_robot/ur_description/urdf/inc/ur_macro.xacro (robot description, xacro)
@@ -325,10 +325,10 @@
     <origin xyz="0 0 0.004" rpy="0 ${-pi/2} ${pi}"/>
   </xacro:soft_robotics_gripper>
-       <!-- <gazebo>
+    <gazebo>
       <plugin name="ros_control" filename="libgazebo_ros_control.so">
         <robotNamespace>/</robotNamespace>
         <robotSimType>gazebo_ros_control/DefaultRobotHWSim</robotSimType>
       </plugin>
-    </gazebo>-->
+    </gazebo>
   </xacro:macro>
 </robot>

File: fmauch_universal_robot/ur_gazebo/urdf/ur_macro.xacro (robot description, xacro)
@@ -81,14 +81,10 @@
       <selfCollide>true</selfCollide>
     </gazebo>
-    <!--
-      Inject Gazebo ROS Control plugin, which allows us to use ros_control
-      controllers to control the virtual robot hw.
-    -->
-    <gazebo>
+    <!--<gazebo>
       <plugin name="ros_control" filename="libgazebo_ros_control.so">
-        <!--robotNamespace>/</robotNamespace-->
-        <!--robotSimType>gazebo_ros_control/DefaultRobotHWSim</robotSimType-->
+        <robotNamespace>/</robotNamespace>
+        <robotSimType>gazebo_ros_control/DefaultRobotHWSim</robotSimType>
       </plugin>
-    </gazebo>
+    </gazebo>-->
   </xacro:macro>
 </robot>

File: soft_robotics/soft_robotics_description/urdf/soft_robotics_gripper.urdf.xacro (robot description, xacro)
@@ -9,5 +9,4 @@
 -->
 <robot name="soft_robotics_gripper" xmlns:xacro="http://www.ros.org/wiki/xacro">
-  <xacro:include filename="$(find soft_robotics_description)/urdf/soft_robotics_trasmission.urdf.xacro" params="" />
   <material name="Grey">
     <color rgba="0.2 0.2 0.2 1" />
@@ -46,5 +45,5 @@
       <parent link="soft_robotics_gripper_base_link" />
       <child link="soft_robotics_left_finger_link1" />
-      <limit effort="0.1" velocity="1" lower="-0.28" upper="0" />
+      <limit effort="1" velocity="1" lower="-0.30" upper="0" />
     </joint>
     <link name="soft_robotics_left_finger_link1">
@@ -72,5 +71,5 @@
       <parent link="soft_robotics_gripper_base_link" />
       <child link="soft_robotics_right_finger_link1" />
-      <limit effort="0.1" velocity="1" lower="-0.28" upper="0" />
+      <limit effort="1" velocity="1" lower="-0.30" upper="0" />
     </joint>
     <link name="soft_robotics_right_finger_link1">
@@ -155,4 +154,23 @@
         <material>Gazebo/Blue</material>
   </gazebo>
+    <!-- TRANSMISSION -->
+    <transmission name="right_finger_trans">
+      <type>transmission_interface/SimpleTransmission</type>
+      <joint name="soft_robotics_gripper_left_finger_joint1">
+        <hardwareInterface>hardware_interface/PositionJointInterface</hardwareInterface>
+      </joint>
+      <actuator name="right_finger_motor">
+        <mechanicalReduction>1</mechanicalReduction>
+      </actuator>
+    </transmission>
+    <transmission name="left_finger_trans">
+      <type>transmission_interface/SimpleTransmission</type>
+      <joint name="soft_robotics_gripper_right_finger_joint1">
+        <hardwareInterface>hardware_interface/PositionJointInterface</hardwareInterface>
+      </joint>
+      <actuator name="${prefix}shoulder_lift_motor">
+        <mechanicalReduction>1</mechanicalReduction>
+      </actuator>
+    </transmission>
   </xacro:macro>
 </robot>
